File: Schematics/DriveAssist_Kicad/DriveAssist_Kicad.kicad_pcb (KiCad board)
At the start: 2 copper layers, 90 x 61 mm, 10 parts, among them J1 APDS 9960, J2 NEO 6M GPS, J3 Speaker, J4 DFP IO, J5 DFP USB, J6 unused, J7 unused_2, U1 DFR0299

Commit message: generated gerber files
Parts:
- added J8: 5V PWR, Connector_PinSocket_2.54mm:PinSocket_1x01_P2.54mm_Vertical, F.Cu at (184.5, 73.0)
- added J9: PWR GND, Connector_PinSocket_2.54mm:PinSocket_1x01_P2.54mm_Vertical, F.Cu at (184.5, 80.5)
- J6: moved to F.Cu
- moved J6 27.4 mm to (147.0, 96.0), turned to 0 degrees
- moved J7 10.0 mm to (147.0, 124.0)
- moved J1 2.83 mm to (185.0, 92.5)
Routing:
- net GND 2: track 0.00 -> 161.7 mm
- net Net-(A1-D2): track 0.00 -> 108.3 mm
- net +5V: track 15.1 -> 98.3 mm
- net Net-(A1-D10): track 0.00 -> 82.3 mm
- net Net-(A1-D11): track 0.00 -> 63.6 mm
- net +3.3V: track 0.00 -> 47.5 mm
- net Net-(A1-D6): track 0.00 -> 33.8 mm
- net Net-(A1-D9): track 37.8 -> 70.6 mm
- net Net-(A1-D5): track 0.00 -> 27.9 mm
- net Net-(A1-D8): track 0.00 -> 24.9 mm
- net Net-(A1-D7): track 0.00 -> 24.7 mm
- net GND 1: track 0.00 -> 18.9 mm
- net Net-(A1-D3): track 0.00 -> 15.3 mm
- net Net-(A1-A5): track 0.00 -> 13.9 mm
- net Net-(A1-D4): track 0.00 -> 13.2 mm
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- added copper zone on B.Cu, net GND 1
Other:
- board size 90 x 61 mm -> 86.5 x 66 mm
- board text added: "5V"
- board text added: "APDS9960"
- board text added: "Driver Assist Version 1.0"
- board text added: "Feb.2026"
- board text added: "GND"
- board text added: "GPS"
- board text added: "Long live Open Source !"
- board text added: "Speaker"
