File: Schematics/DriveAssist_Kicad/DriveAssist_Kicad.kicad_sch (KiCad schematic)
At the start: 12 parts, among them J1 APDS 9960, J2 NEO 6M GPS, J3 Speaker, J4 DFP IO, J5 DFP USB, J6 unused, J7 unused_2, J8 Conn_01x01_Socket, J9 PWR GND, U1 DFR0299

Commit message: generated gerber files
Parts:
- J8: value Conn_01x01_Socket -> 5V PWR; footprint (none) -> Connector_PinSocket_2.54mm:PinSocket_1x01_P2.54mm_Vertical
- J9: footprint (none) -> Connector_PinSocket_2.54mm:PinSocket_1x01_P2.54mm_Vertical
Connections:
- net +5V: now also J8.1 (Pin_1)
- no-connect marks 38 -> 40
Other:
- moved on the sheet: J8
Changed lines of the file:
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@@
+	)
+	(junction
+		(at 130.81 57.15)
+		(diameter 0)
+		(color 0 0 0 0)
 	)
 	(junction
@@
 	)
 	(no_connect
+		(at 130.81 49.53)
+	)
+	(no_connect
 		(at 173.99 92.71)
 	)
@@
 	)
 	(no_connect
+		(at 123.19 118.11)
+	)
+	(no_connect
 		(at 63.5 102.87)
 	)
@@
 	(wire
 		(pts
-			(xy 125.73 57.15) (xy 151.13 57.15)
+			(xy 125.73 57.15) (xy 130.81 57.15)
 		)
 		(stroke
@@
 	(wire
 		(pts
+			(xy 130.81 54.61) (xy 130.81 57.15)
+		)
+		(stroke
+			(width 0)
+			(type default)
+		)
+	)
+	(wire
+		(pts
 			(xy 125.73 67.31) (xy 123.19 67.31)
 		)
@@
 		(pts
 			(xy 168.91 54.61) (xy 168.91 87.63)
+		)
+		(stroke
+			(width 0)
+			(type default)
+		)
+	)
+	(wire
+		(pts
+			(xy 130.81 57.15) (xy 151.13 57.15)
 		)
 		(stroke
@@
 	(symbol
 		(lib_id "Connector:Conn_01x01_Socket")
-		(at 135.89 53.34 0)
+		(at 130.81 49.53 90)
 		(unit 1)
 		(exclude_from_sim no)
@@
 		(fields_autoplaced yes)
 		(property "Reference" "J8"
-			(at 137.16 52.0699 0)
-			(effects
-				(font
-					(size 1.27 1.27)
-				)
-				(justify left)
-			)
-		)
-		(property "Value" "Conn_01x01_Socket"
-			(at 137.16 54.6099 0)
-			(effects
-				(font
-					(size 1.27 1.27)
-				)
-				(justify left)
-			)
-		)
-		(property "Footprint" ""
-			(at 135.89 53.34 0)
+			(at 132.08 48.8949 90)
+			(effects
+				(font
+					(size 1.27 1.27)
+				)
+				(justify right)
+			)
+		)
+		(property "Value" "5V PWR"
+			(at 132.08 51.4349 90)
+			(effects
+				(font
+					(size 1.27 1.27)
+				)
+				(justify right)
+			)
+		)
+		(property "Footprint" "Connector_PinSocket_2.54mm:PinSocket_1x01_P2.54mm_Vertical"
+			(at 130.81 49.53 0)
 			(effects
 				(font
@@
 		)
 		(property "Datasheet" "~"
-			(at 135.89 53.34 0)
+			(at 130.81 49.53 0)
 			(effects
 				(font
@@
 		)
 		(property "Description" "Generic connector, single row, 01x01, script generated"
-			(at 135.89 53.34 0)
+			(at 130.81 49.53 0)
 			(effects
 				(font
@@
 			)
 		)
-		(property "Footprint" ""
+		(property "Footprint" "Connector_PinSocket_2.54mm:PinSocket_1x01_P2.54mm_Vertical"
 			(at 123.19 118.11 0)
 			(effects
